Commit message: Fix references to missing turtlebot3_gazebo package

File: lab2_2026/src/bringup/urdf/turtlebot3_burger.urdf (robot description, URDF)
Before this commit: robot turtlebot3_burger, 7 links, 6 joints
Links:
- link base_link: geometry collision box size=0.140 0.140 0.143; visual mesh filename=package://bringup/models/turtlebot3_common/meshes/burger_ba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 scale=0.001 0.001 0.001
- link base_scan: geometry collision cylinder length=0.0315 radius=0.055; visual mesh filename=package://bringup/models/turtlebot3_common/meshes/lds.dae scale=0.001 0.001 0.001
- link wheel_left_link: geometry collision cylinder length=0.018 radius=0.033; visual mesh filename=package://bringup/models/turtlebot3_common/meshes/tire.dae scale=0.001 0.001 0.001
- link wheel_right_link: geometry collision cylinder length=0.018 radius=0.033; visual mesh filename=package://bringup/models/turtlebot3_common/meshes/tire.dae scale=0.001 0.001 0.001

File: lab2_2026/src/bringup/urdf/turtlebot3_waffle.urdf (robot description, URDF)
Before this commit: robot turtlebot3_waffle, 13 links, 12 joints
Links:
- link base_link: geometry collision box size=0.266 0.266 0.094; visual mesh filename=package://bringup/models/turtlebot3_common/meshes/waffle_ba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 scale=0.001 0.001 0.001
- link base_scan: geometry collision cylinder length=0.0315 radius=0.055; visual mesh filename=package://bringup/models/turtlebot3_common/meshes/lds.dae scale=0.001 0.001 0.001
- link camera_link: geometry collision box size=0.012 0.132 0.020; visual mesh filename=package://bringup/models/turtlebot3_common/meshes/r200.dae
- link wheel_left_link: geometry collision cylinder length=0.018 radius=0.033; visual mesh filename=package://bringup/models/turtlebot3_common/meshes/tire.dae scale=0.001 0.001 0.001
- link wheel_right_link: geometry collision cylinder length=0.018 radius=0.033; visual mesh filename=package://bringup/models/turtlebot3_common/meshes/tire.dae scale=0.001 0.001 0.001
